Commit message: made changes to several files and changed package name

File: urdf/ar2019.urdf.xacro (robot description, xacro)
@@ -16,5 +16,5 @@
       <origin xyz="0 0 0" rpy="0 1.57 1.57"/>
       <geometry>
-        <mesh filename="package://waffle_pick_place/worlds/artag.dae"/>
+        <mesh filename="package://waffle_slam/worlds/artag.dae"/>
       </geometry>
     </visual>
